File: Fan_Controller.kicad_pcb (KiCad board)
At the start: 4 copper layers, 35 x 35 mm, 44 parts, among them J1 Conn_02x02_Odd_Even, J2 Conn_01x03_MountingPin, J3 Conn_01x04_MountingPin, J4 Conn_01x06, Q1 AO3400A, U1 LM51571, U2 ESP32-C6-MINI-1, U3 RT9193-33GB, U4 MAX31865xTP, U5 TMP112xxDRL

Commit message: Workflow Update
Parts:
- J1: value Conn_02x02_Odd_Even -> DF11-4DP-2DSA
- J2: value Conn_01x03_MountingPin -> 53047-0310
- J3: value Conn_01x04_MountingPin -> 53047-0510
- J4: value Conn_01x06 -> TP_01x06_P2.54

Commit message: Update
Parts:
- added R10: 5.1K, Resistor_SMD:R_0402_1005Metric, F.Cu at (108.9, 92.8)
- added R11: 5.1K, Resistor_SMD:R_0402_1005Metric, F.Cu at (108.9, 93.9)
- added TP1: TestPoint, TestPoint:TestPoint_Pad_D1.0mm, B.Cu at (100.4, 74.4)
- added TP2: TestPoint, TestPoint:TestPoint_Pad_D1.0mm, B.Cu at (102.6, 74.4)
- R6: value 100K -> 10K
Connections:
- J4 pad 5: /TXD -> /D-
- J4 pad 6: /RXD -> /D+
- U2 pad 17: /SCL -> /D-
- U2 pad 18: /SDA -> /D+
- U2 pad 19: unconnected-(U2-IO14-Pad19) -> /SCL
- U2 pad 20: unconnected-(U2-IO15-Pad20) -> /SDA
Routing:
- net /D-: track 0.00 -> 10.9 mm, vias 0 -> 1
- net /D+: track 0.00 -> 10.3 mm, vias 0 -> 1
- net /RXD: track 8.24 -> 2.12 mm, vias 0 -> 1
- net /TXD: track 6.46 -> 2.05 mm, vias 0 -> 1
- net /SDA: track 17.3 -> 21.2 mm
- net /SCL: track 15.8 -> 18.6 mm
- net +3V3: track 7.75 -> 8.77 mm, vias 10 -> 11
Other:
- board text added: "Designed by Acha Fan_Controller ${BRANCH}-${SHORT_SHA}-${CURRENT_DATE}"
