File: Fan_Controller.kicad_sch (KiCad schematic)
At the start: 52 parts, among them J1 Conn_02x02_Odd_Even, J2 Conn_01x03_MountingPin, J3 Conn_01x04_MountingPin, J4 Conn_01x06, Q1 AO3400A, U1 LM51571, U101 TPS61093, U2 ESP32-C6-MINI-1, U3 RT9193-33GB, U4 MAX31865xTP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

Commit message: Workflow Update
Parts:
- J1: value Conn_02x02_Odd_Even -> DF11-4DP-2DSA
- J2: value Conn_01x03_MountingPin -> 53047-0310
- J3: value Conn_01x04_MountingPin -> 53047-0510
- J4: value Conn_01x06 -> TP_01x06_P2.54; now left out of the parts list
Other:
- moved on the sheet: C1, C11, C15, C16, C17, C2, C3, C4, C5, C6, C7, C8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

Commit message: Update
Parts:
- added R10, R11: 5.1K, Resistor_SMD:R_0402_1005Metric, symbol Device:R_Small
- added TP1, TP2: TestPoint, TestPoint:TestPoint_Pad_D1.0mm, symbol Connector:TestPoint
- R6: value 100K -> 10K
Connections:
- net +3V3: now also R10.1, R11.1
- net RXD: now also TP2.1; no longer J4.6 (Pin_6)
- net SCL: now also U2.19 (IO14), R11.2; no longer U2.17 (IO12)
- net SDA: now also U2.20 (IO15), R10.2; no longer U2.18 (IO13)
- net TXD: now also TP1.1; no longer J4.5 (Pin_5)
- new net D+: J4.6 (Pin_6), U2.18 (IO13)
- new net D-: J4.5 (Pin_5), U2.17 (IO12)
- no-connect marks 3 -> 11
